File: Hardware/Rpi Servo Stepper/Cartev1.sch (EAGLE design)
At the start: 8 parts

Commit message: Hardware V2 PROD
Version ITEAD Studio Production
Parts:
- removed LM2575T-ADJ: LM2575T-ADJ, LM2575T:LM2575T-ADJ
- removed U$3: HEADER_25*2.54MM, Headers:HEADER_252.54MM
- removed U$4: HEADER_232.54MM, Headers:HEADER_232.54MM
- added +12V, GND: (no value), wirepad:3,81/1,4
- added C1: 100uf, rcl:CPOL-EUE
- added C2: 1000uF, rcl:CPOL-EUG
- added D2: (no value), diode:SCHOTTKY-DIODESMC
- added J1: 1X2-3.5MM, adafruit (2):1X2-3.5MM
- added L1: SDR2207, bourns-inductor:SDR2207
- added LM1: LM2576-5V, linear:LM2596S
- added SJ1, SJ2, SJ3, SJ4: SOLDERJUMPERTRACE, SparkFun-Passives:SOLDERJUMPERTRACE
- added TP1: TPTP10SQ, testpad:TPTP10SQ
- D1: value VS-11DQ06 -> (none); device adafruit:SCHOTTKY-DIODEDO41 -> diode:SCHOTTKY-DIODESMC
- U$2: value HEADER_252.54MM -> CONNECTEUR_RPI; device Headers:HEADER_252.54MM -> Rpi:CONNECTEUR_RPI
Connections:
- new net +5V: C2.+, L1.2, LB1948MC-AH.VCC, LM1.FB, SERVO.2, TP1.TP, U$2.5V_1, U$2.5V_2
- new net N$10: LB1948MC-AH.IN4, SJ4.1
- new net N$11: SERVO.1, U$2.GPIO25
- new net N$12: SJ1.2, U$2.GPIO21/GPIO27
- new net N$13: SJ2.2, U$2.GPIO22
- new net N$14: SJ3.2, U$2.GPIO23
- new net N$15: SJ4.2, U$2.GPIO24
- new net N$6: D2.C, L1.1, LM1.OUT
- new net N$7: LB1948MC-AH.IN1, SJ1.1
- new net N$8: LB1948MC-AH.IN2, SJ2.1
- new net N$9: LB1948MC-AH.IN3, SJ3.1
- new net VDD: C1.+, D1.C, LM1.IN
- net GND: now also C1.-, C2.-, D2.A, GND.P, J1.1, LM1.EN, LM1.GND, LM1.GND@1, SERVO.3, U$2.GND_1, U$2.GND_2, U$2.GND_3, U$2.GND_4, U$2.GND_5; no longer LM2575T-ADJ.GND
- net N$5: now also +12V.P, D1.A, J1.2; no longer LB1948MC-AH.VCC, LM2575T-ADJ.VIN
Other:
- moved on the sheet: D1, LB1948MC-AH, SERVO
